File: paperkb.kicad_pcb (KiCad board)
At the start: 2 copper layers, 128 parts, among them SW1 KS33_SW_solder, SW10 KS33_SW_solder, SW11 KS33_SW_solder, SW12 KS33_SW_solder, SW13 KS33_SW_solder, SW14 KS33_SW_solder, SW15 KS33_SW_solder, SW16 KS33_SW_solder, SW17 KS33_SW_solder, SW18 KS33_SW_solder, SW19 KS33_SW_solder, SW2 KS33_SW_solder, SW20 KS33_SW_solder, SW21 KS33_SW_solder, SW22 KS33_SW_solder, SW23 KS33_SW_solder, SW24 KS33_SW_solder, SW25 KS33_SW_solder, SW26 KS33_SW_solder, SW27 KS33_SW_solder, SW28 KS33_SW_solder, SW29 KS33_SW_solder, SW3 KS33_SW_solder, SW30 KS33_SW_solder, SW31 KS33_SW_solder, SW32 KS33_SW_solder, SW33 KS33_SW_solder, SW34 KS33_SW_solder, SW35 KS33_SW_solder, SW36 KS33_SW_solder, SW37 KS33_SW_solder, SW38 KS33_SW_solder, SW39 KS33_SW_solder, SW4 KS33_SW_solder, SW40 KS33_SW_solder, SW41 KS33_SW_solder, SW42 KS33_SW_solder, SW43 KS33_SW_solder, SW44 KS33_SW_solder, SW45 KS33_SW_solder, SW46 KS33_SW_solder, SW47 KS33_SW_solder, SW48 KS33_SW_solder, SW49 KS33_SW_solder, SW5 KS33_SW_solder, SW50 KS33_SW_solder, SW51 KS33_SW_solder, SW52 KS33_SW_solder, SW53 KS33_SW_solder, SW54 KS33_SW_solder, SW55 KS33_SW_solder, SW56 KS33_SW_solder, SW57 KS33_SW_solder, SW58 KS33_SW_solder, SW59 KS33_SW_solder, SW6 KS33_SW_solder, SW60 KS33_SW_solder, SW61 KS33_SW_solder, SW62 KS33_SW_solder, SW63 KS33_SW_solder, SW64 KS33_SW_solder, SW7 KS33_SW_solder, SW8 KS33_SW_solder, SW9 KS33_SW_solder

Commit message: schematic finished?
Parts:
- added C1: 1uF, Capacitor_SMD:C_0603_1608Metric, F.Cu at (160.5, 169.3)
- added C10: 100nF, Capacitor_SMD:C_0603_1608Metric, F.Cu at (164.5, 176.8)
- added C11: 100nF, Capacitor_SMD:C_0603_1608Metric, F.Cu at (164.5, 179.3)
- added C12: 100nF, Capacitor_SMD:C_0603_1608Metric, F.Cu at (164.5, 181.8)
- added C13: 100nF, Capacitor_SMD:C_0603_1608Metric, F.Cu at (168.5, 169.3)
- added C14: 100nF, Capacitor_SMD:C_0603_1608Metric, F.Cu at (168.5, 171.8)
- added C15: 1uF, Capacitor_SMD:C_0603_1608Metric, F.Cu at (168.5, 174.3)
- added C16: 1uF, Capacitor_SMD:C_0603_1608Metric, F.Cu at (168.5, 176.8)
- added C17: 100nF, Capacitor_SMD:C_0603_1608Metric, F.Cu at (168.5, 179.3)
- added C2: 1uF, Capacitor_SMD:C_0603_1608Metric, F.Cu at (160.5, 171.8)
- added C3: 15pF, Capacitor_SMD:C_0603_1608Metric, F.Cu at (160.5, 174.3)
- added C4: 15pF, Capacitor_SMD:C_0603_1608Metric, F.Cu at (160.5, 176.8)
- added C5: 100nF, Capacitor_SMD:C_0603_1608Metric, F.Cu at (160.5, 179.3)
- added C6: 100nF, Capacitor_SMD:C_0603_1608Metric, F.Cu at (160.5, 181.8)
- added C7: 100nF, Capacitor_SMD:C_0603_1608Metric, F.Cu at (164.5, 169.3)
- added C8: 100nF, Capacitor_SMD:C_0603_1608Metric, F.Cu at (164.5, 171.8)
- added C9: 100nF, Capacitor_SMD:C_0603_1608Metric, F.Cu at (164.5, 174.3)
- added J1: USB_C_Receptacle_USB2.0_16P, Connector_USB:USB_C_Receptacle_HRO_TYPE-C-31-M-12, F.Cu at (168.9, 196.5)
- added J2: Conn_01x12, FallCTF:FPC-SMD_AFC01-S12FCA-00, F.Cu at (169.0, 185.6)
- added J3: Conn_01x04, Connector_PinHeader_2.54mm:PinHeader_1x04_P2.54mm_Vertical, F.Cu at (160.8, 185.4)
- added Q1: AO3400A, Package_TO_SOT_SMD:SOT-23, F.Cu at (187.8, 185.3)
- added R1: 10k, Resistor_SMD:R_0603_1608Metric, F.Cu at (168.5, 181.8)
- added R10: 10k, Resistor_SMD:R_0603_1608Metric, F.Cu at (176.5, 174.3)
- added R11: 10k, Resistor_SMD:R_0603_1608Metric, F.Cu at (176.5, 176.8)
- added R12: 220, Resistor_SMD:R_0603_1608Metric, F.Cu at (176.5, 179.3)
- added R15: 100k, Resistor_SMD:R_0603_1608Metric, F.Cu at (176.5, 181.8)
- added R2: 1K, Resistor_SMD:R_0603_1608Metric, F.Cu at (172.5, 169.3)
- added R3: 1k, Resistor_SMD:R_0603_1608Metric, F.Cu at (172.5, 171.8)
- added R4: 10k, Resistor_SMD:R_0603_1608Metric, F.Cu at (172.5, 174.3)
- added R5: 5.1k, Resistor_SMD:R_0603_1608Metric, F.Cu at (172.5, 176.8)
- added R6: 5.1k, Resistor_SMD:R_0603_1608Metric, F.Cu at (172.5, 179.3)
- added R7: 27, Resistor_SMD:R_0603_1608Metric, F.Cu at (172.5, 181.8)
- added R8: 27, Resistor_SMD:R_0603_1608Metric, F.Cu at (176.5, 169.3)
- added R9: 10, Resistor_SMD:R_0603_1608Metric, F.Cu at (176.5, 171.8)
- added SW65: SW_Push, Button_Switch_SMD:SW_Push_1P1T_XKB_TS-1187A, F.Cu at (182.8, 171.3)
- added SW66: SW_Push, Button_Switch_SMD:SW_Push_1P1T_XKB_TS-1187A, F.Cu at (182.8, 178.0)
- added U1: RP2040, Package_DFN_QFN:QFN-56-1EP_7x7mm_P0.4mm_EP3.2x3.2mm, F.Cu at (180.0, 194.7)
- added U2: AP2112K-3.3, Package_TO_SOT_SMD:SOT-23-5, F.Cu at (187.2, 197.0)
- added U3: W25Q128JVS, Package_SO:SOIC-8_5.3x5.3mm_P1.27mm, F.Cu at (180.2, 186.6)
- added Y1: 12MHz, Crystal:Crystal_SMD_3225-4Pin_3.2x2.5mm, F.Cu at (187.3, 192.3)
- SW1, SW10, SW11, SW12, SW13, SW14, SW15, SW16, SW17, SW18, SW19, SW2, SW20, SW21, SW22, SW23, SW24, SW25, SW26, SW27, SW28, SW29, SW3, SW30, SW31, SW32, SW33, SW34, SW35, SW36, SW37, SW38, SW39, SW4, SW40, SW41, SW42, SW43, SW44, SW45, SW46, SW47, SW48, SW49, SW5, SW50, SW51, SW52, SW53, SW54, SW55, SW56, SW57, SW58, SW59, SW6, SW60, SW61, SW62, SW63, SW64, SW7, SW8, SW9: footprint marbastlib-xp-gateron_lp:SW_KS33_1u -> PCM_marbastlib-xp-gateron_lp:SW_KS33_1u
Connections:
- SW14 pad 1: COL12 -> COL13
- SW28 pad 1: COL12 -> COL13

Commit message: assign jlcpcb parts
Parts:
- C3, C4: value 15pF -> 30pF
- R2: value 1K -> 1k
