File: paperkb.kicad_sch (KiCad schematic)
At the start: 164 parts, among them J1 USB_C_Receptacle_USB2.0_16P, J2 Conn_01x12, Q1 AO3400A, SW1 KS33_SW_solder, SW10 KS33_SW_solder, SW11 KS33_SW_solder, SW12 KS33_SW_solder, SW13 KS33_SW_solder, SW14 KS33_SW_solder, SW15 KS33_SW_solder, SW16 KS33_SW_solder, SW17 KS33_SW_solder, SW18 KS33_SW_solder, SW19 KS33_SW_solder, SW2 KS33_SW_solder, SW20 KS33_SW_solder, SW21 KS33_SW_solder, SW22 KS33_SW_solder, SW23 KS33_SW_solder, SW24 KS33_SW_solder, SW25 KS33_SW_solder, SW26 KS33_SW_solder, SW27 KS33_SW_solder, SW28 KS33_SW_solder, SW29 KS33_SW_solder, SW3 KS33_SW_solder, SW30 KS33_SW_solder, SW31 KS33_SW_solder, SW32 KS33_SW_solder, SW33 KS33_SW_solder, SW34 KS33_SW_solder, SW35 KS33_SW_solder, SW36 KS33_SW_solder, SW37 KS33_SW_solder, SW38 KS33_SW_solder, SW39 KS33_SW_solder, SW4 KS33_SW_solder, SW40 KS33_SW_solder, SW41 KS33_SW_solder, SW42 KS33_SW_solder, SW43 KS33_SW_solder, SW44 KS33_SW_solder, SW45 KS33_SW_solder, SW46 KS33_SW_solder, SW47 KS33_SW_solder, SW48 KS33_SW_solder, SW49 KS33_SW_solder, SW5 KS33_SW_solder, SW50 KS33_SW_solder, SW51 KS33_SW_solder, SW52 KS33_SW_solder, SW53 KS33_SW_solder, SW54 KS33_SW_solder, SW55 KS33_SW_solder, SW56 KS33_SW_solder, SW57 KS33_SW_solder, SW58 KS33_SW_solder, SW59 KS33_SW_solder, SW6 KS33_SW_solder, SW60 KS33_SW_solder, SW61 KS33_SW_solder, SW62 KS33_SW_solder, SW63 KS33_SW_solder, SW64 KS33_SW_solder, SW65 SW_Push, SW66 SW_Push, SW7 KS33_SW_solder, SW8 KS33_SW_solder, SW9 KS33_SW_solder, U1 RP2040, U2 AP2112K-3.3, U3 W25Q128JVS, Y1 12MHz

Commit message: schematic finished?
Parts:
- added C17: 100nF, Capacitor_SMD:C_0603_1608Metric, symbol Device:C_Small
- added J3: Conn_01x04, Connector_PinHeader_2.54mm:PinHeader_1x04_P2.54mm_Vertical, symbol Connector_Generic:Conn_01x04
- added R12: 220, Resistor_SMD:R_0603_1608Metric, symbol Device:R_Small
- added R15: 100k, Resistor_SMD:R_0603_1608Metric, symbol Device:R_Small
- C1, C10, C11, C12, C13, C14, C15, C16, C2, C3, C4, C5, C6, C7, C8, C9: footprint (none) -> Capacitor_SMD:C_0603_1608Metric
- J1: footprint (none) -> Connector_USB:USB_C_Receptacle_HRO_TYPE-C-31-M-12
- R1, R10, R11, R2, R3, R4, R5, R6, R7, R8, R9: footprint (none) -> Resistor_SMD:R_0603_1608Metric
- SW65, SW66: footprint (none) -> Button_Switch_SMD:SW_Push_1P1T_XKB_TS-1187A
- Y1: footprint (none) -> Crystal:Crystal_SMD_3225-4Pin_3.2x2.5mm
Connections:
- net +3V3: now also C17.2, J3.4 (Pin_4)
- net GND: now also Q1.2 (S), C17.1, J3.1 (Pin_1), R15.2
- net TFT_CS: now also U1.37 (GPIO25)
- net TFT_DC: now also U1.34 (GPIO22)
- net TFT_MOSI: now also U1.39 (GPIO27/ADC1)
- net TFT_RST: now also U1.35 (GPIO23)
- net TFT_SCK: now also U1.38 (GPIO26/ADC0)
- net XOUT: no longer C4.1
- net at R2.1, Y1.3: now also C4.1
- net at Q1.1 (G): now also R12.2, R15.1
- net TFT_LEDK: now reaches Q1.3 (D)
- net TFT_LEDK: now also J2.8 (Pin_8)
- net SWCLK: now reaches U1.24 (SWCLK)
- net SWCLK: now also J3.3 (Pin_3)
- net SWDIO: now reaches U1.25 (SWDIO)
- net SWDIO: now also J3.2 (Pin_2)
- net TFT_BL: now reaches U1.36 (GPIO24)
- net TFT_BL: now also R12.1
- no-connect marks 0 -> 7
Other:
- note added: "Debug"
- note added: "Display Connector"
- moved on the sheet: C4, Q1, R2

Commit message: assign jlcpcb parts
Parts:
- C3, C4: value 15pF -> 30pF
- R2: value 1K -> 1k
Changed lines of the file:
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@@
 			)
 		)
-		(property "Value" "15pF"
+		(property "Value" "30pF"
 			(at 166.37 223.5262 0)
 			(show_name no)
@@
 			)
 		)
-		(property "Value" "15pF"
+		(property "Value" "30pF"
 			(at 182.88 222.2562 0)
 			(show_name no)
@@
 			)
 		)
-		(property "Value" "1K"
+		(property "Value" "1k"
 			(at 186.69 213.36 90)
 			(show_name no)
